Commit message: Updated A* algorithm

File: simulation/objects/wall_with_door.urdf (robot description, URDF)
Before this commit: robot wall_with_door, 4 links, 3 joints
Links:
- removed link base_link
- removed link left_wall
- removed link right_wall
- removed link top_wall
- added link wall_with_door_link, mass 45.0; collision box size=2 0.2 1; collision box size=7.5 0.2 3
Joints:
- removed joint joint_left
- removed joint joint_right
- removed joint joint_top_wall
