Commit message: Added Motion plot

File: simulation/objects/wall.urdf (robot description, URDF)
Before this commit: robot wall, 1 links, 0 joints
Links:
- link wall_link: geometry collision box size=16.5 0.2 3; visual box size=16.5 0.2 3

Commit message: Updated wall.urdf

File: simulation/objects/wall.urdf (robot description, URDF)
Before this commit: robot wall, 1 links, 0 joints
Links:
- link wall_link: geometry collision box size=16.2 0.2 3; visual box size=16.2 0.2 3
